File: TAStable.kicad_sch (KiCad schematic)
At the start: 12 parts, among them J1 Conn_01x06_Pin, U1 74HCT1G04, U2 CS2300-CP, U3 74LVC1G14

Commit message: cleanups
Other:
- moved on the sheet: C1, C3, J1, R1, R2, U3

Commit message: code!
Parts:
- added C6: 22uF Tantalum, Capacitor_SMD:C_1206_3216Metric, symbol Device:C_Polarized_US
- added C7: 1uF, Capacitor_SMD:C_0603_1608Metric, symbol Device:C
- added C8: 100nF, Capacitor_SMD:C_0603_1608Metric, symbol Device:C
- added J2: ICSP, Connector_PinSocket_2.54mm:PinSocket_1x05_P2.54mm_Vertical, symbol Connector:Conn_01x05_Pin
- added U4: PIC16LF15313, Package_SO:SOIC-8_3.9x4.9mm_P1.27mm, symbol MCU_Microchip_PIC12:PIC12F1501-IMS
- added U6: AZ1117-3.3, Package_TO_SOT_SMD:SOT-89-3, symbol Regulator_Linear:AZ1117-3.3
Connections:
- net I2C_SDA is gone; now on net I2C_SCL: J1.3 (Pin_3), R1.2, U2.10 (SDA/CDIN)
- net +3.3V: now also C6.1, C7.1, C8.1, J2.2 (Pin_2), U4.1 (VDD), U6.2 (VO); no longer C5.1, J1.1 (Pin_1)
- net GND: now also C6.2, C7.2, C8.2, J2.3 (Pin_3), U4.8 (VSS), U6.1 (GND)
- net I2C_SCL: now also J2.5 (Pin_5), U4.5 (RA2), U4.6 (RA1)
- new net +5V: C5.1, J1.1 (Pin_1), U6.3 (VI)
- new net ICSPDAT: J2.4 (Pin_4), U4.7 (RA0)
- new net MCLR: J2.1 (Pin_1), U4.4 (RA3)
Other:
- note added: "Jumper MCLR to 3.3v when programmed"
- moved on the sheet: C1, C3, U3

Commit message: 5v output buffer
Connections:
- net +3.3V: no longer C4.1, U1.5 (VCC)
- net +5V: now also C4.1, U1.5 (VCC)
Changed lines of the file:
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@@
+    )
+  )
+  (symbol (lib_id "power:+5V") (at 172.72 63.5 0) (unit 1)
+    (in_bom yes) (on_board yes) (dnp no) (fields_autoplaced)
+    (property "Reference" "#PWR09" (at 172.72 67.31 0)
+      (effects (font (size 1.27 1.27)) hide)
+    )
+    (property "Value" "+5V" (at 172.72 59.69 0)
+      (effects (font (size 1.27 1.27)))
+    )
+    (property "Footprint" "" (at 172.72 63.5 0)
+      (effects (font (size 1.27 1.27)) hide)
+    )
+    (property "Datasheet" "" (at 172.72 63.5 0)
+      (effects (font (size 1.27 1.27)) hide)
+    )
+    (pin "1")
+    (instances
+      (project "TAStable"
+        (path "/e6d4ff55-0377-40c6-85e0-bfd48c6c6235"
+          (reference "#PWR09") (unit 1)
+        )
+      )
     )
   )
@@
         )
       )
-    )
-  )
-  (symbol (lib_id "power:+3.3V") (at 172.72 63.5 0) (unit 1)
-    (in_bom yes) (on_board yes) (dnp no) (fields_autoplaced)
-    (property "Reference" "#PWR09" (at 172.72 67.31 0)
-      (effects (font (size 1.27 1.27)) hide)
-    )
-    (property "Value" "+3.3V" (at 172.72 59.69 0)
-      (effects (font (size 1.27 1.27)))
-    )
-    (property "Footprint" "" (at 172.72 63.5 0)
-      (effects (font (size 1.27 1.27)) hide)
-    )
-    (property "Datasheet" "" (at 172.72 63.5 0)
-      (effects (font (size 1.27 1.27)) hide)
-    )
-    (pin "1")
-    (instances
-      (project "TAStable"
-        (path "/e6d4ff55-0377-40c6-85e0-bfd48c6c6235"
-          (reference "#PWR09") (unit 1)
-        )
-      )

Commit message: more pics + cleanups
Parts:
- J1: value Conn_01x06_Pin -> IN/OUT
Connections:
- net 24MHz_OUT: now also J1.6 (Pin_6), U1.4
- net I2C_SCL: no longer J1.3 (Pin_3), R1.2, U2.10 (SDA/CDIN), U4.5 (RA2)
- new net I2C_SDA: J1.3 (Pin_3), R1.2, U2.10 (SDA/CDIN), U4.5 (RA2)
Other:
- moved on the sheet: C3, C5, C6, C8, J1, J2, R1, R2, U6

Commit message: schematic
Other:
- moved on the sheet: C4, C5, C6, J1, J2, U6

Commit message: v2
Parts:
- removed C5, C7: 1uF, Capacitor_SMD:C_0603_1608Metric, symbol Device:C
- removed C6: 22uF Tantalum, Capacitor_SMD:C_1206_3216Metric, symbol Device:C_Polarized_US
- removed J1: IN/OUT, Connector_PinHeader_2.54mm:PinHeader_1x06_P2.54mm_Horizontal, symbol Connector:Conn_01x06_Pin
- removed U2: CS2300-CP, Package_SO:MSOP-10_3x3mm_P0.5mm, symbol Timer_PLL:CS2000-CP
- removed U3: 74LVC1G14, Package_TO_SOT_SMD:SOT-353_SC-70-5, symbol 74xGxx:74LVC1G14
- removed U6: AZ1117-3.3, Package_TO_SOT_SMD:SOT-89-3, symbol Regulator_Linear:AZ1117-3.3
- added C5: 22uF Tantalum, Capacitor_SMD:C_1206_3216Metric, symbol Device:C_Polarized_US
- added C9: 100nF, Capacitor_SMD:C_0603_1608Metric, symbol Device:C
- added J1: Conn_01x08, symbol Connector_Generic:Conn_01x08
- added U2: Si5351A-B-GT, Package_SO:MSOP-10_3x3mm_P0.5mm, symbol Oscillator:Si5351A-B-GT
- added U3: 74HCT1G04, Package_TO_SOT_SMD:SOT-353_SC-70-5, symbol 74xGxx:74AHCT1G04
- added U5: AZ1117-3.3, Package_TO_SOT_SMD:SOT-89-3, symbol Regulator_Linear:AZ1117-3.3
- added U6: 74HCT74, symbol 74xx:74HC74
- added Y2: 25MHz, symbol Device:Crystal_GND24_Small
- C2: value 100nF -> 1uF
Connections:
- net ICSPDAT is gone; now on net RESET_IN: J2.4 (Pin_4), U4.7 (RA0)
- net +3.3V: now also C1.1, C5.1, U2.1 (VDD), U2.7 (VDDO), U5.2 (VO); no longer C2.1
- net +5V: now also C2.1, C9.1, J1.1 (Pin_1), U3.5 (VCC), U5.3 (VI)
- net 24MHz_OUT: now also J1.8 (Pin_8), U3.4; no longer U1.4
- net GND: now also C1.2, C5.2, C9.2, J1.2 (Pin_2), U2.8 (GND), U3.3 (GND), U5.1 (GND), Y2.2, Y2.4; no longer C1.1
- net I2C_SCL: now also J1.4 (Pin_4), U2.4 (SCL)
- net I2C_SDA: now also J1.3 (Pin_3), U2.5 (SDA)
- net CLK0: now reaches U1.2
- net CLK0: now also U2.10 (CLK0)
- net RESET_IN: now reaches R3.2
- net RESET_IN: now also J1.5 (Pin_5)
- net at U4.2 (RA5): now also U6.1 (~{R})
- net at U4.3 (RA4): now also U6.2 (D)
- new net: U2.2 (XA), Y2.3
- new net: U2.3 (XB), Y2.1
- new net: U2.9 (CLK1), U6.3 (C)
- new net 21MHz_OUT: J1.7 (Pin_7), U1.4
- new net CLK2: U2.6 (CLK2), U3.2
- new net RESET_OUT: J1.6 (Pin_6), U6.5 (Q)
Other:
- moved on the sheet: C4, C8, J2, R1, R2, U1, U4
