File: TAStable.kicad_sch (KiCad schematic)
At the start: 19 parts, among them J1 Conn_01x08, J2 ICSP, U1 74HCT1G04, U2 Si5351A-B-GT, U3 74HCT1G04, U4 PIC16LF15313, U5 AZ1117-3.3, U6 74HCT74, Y2 25MHz

Commit message: fixes
Parts:
- added C6: 100nF, Capacitor_SMD:C_0603_1608Metric, symbol Device:C
- added unit 3 of U6
- added unit 2 of U6
- J1: footprint (none) -> Connector_PinHeader_2.54mm:PinHeader_1x08_P2.54mm_Vertical
- U6: footprint (none) -> Package_SO:TSSOP-14_4.4x5mm_P0.65mm
- Y2: footprint (none) -> Crystal:Crystal_SMD_Abracon_ABM8G-4Pin_3.2x2.5mm
Connections:
- net +5V: now also C6.1, U6.10 (~{S}), U6.13 (~{R}), U6.14 (VCC)
- net GND: now also C6.2, U6.11 (C), U6.12 (D), U6.7 (GND)
- net CLK1: now reaches U2.9 (CLK1), U6.3 (C)
Other:
- moved on the sheet: C1, C3, J2, Y2

Commit message: andy finally learns FPGA programming
Parts:
- removed C4, C9: 100nF, Capacitor_SMD:C_0603_1608Metric, symbol Device:C
- removed U1, U3: 74HCT1G04, Package_TO_SOT_SMD:SOT-353_SC-70-5, symbol 74xGxx:74AHCT1G04
- added U1: 74HCT00, symbol 74xx:74HCT00
- added U3: 74HCT74, Package_SO:TSSOP-14_4.4x5mm_P0.65mm, symbol 74xx:74HC74
Connections:
- net 21MHz_OUT: now also U1.3
- net GND: now also U3.11 (C), U3.12 (D); no longer U6.11 (C), U6.12 (D)
- net RESET_OUT: now also U6.9 (Q); no longer U6.5 (Q)
- net at U6.8 (~{Q}): now also U3.13 (~{R})
- net at U6.2 (D): no longer U4.3 (RA4)
- net SMPWR: now reaches U6.4 (~{S})
- net SMPWR: now also U3.10 (~{S})
- net CLK0: no longer names the net of U2.10 (CLK0)
- net CLK0: now also U1.1, U1.2
- net CLK1: no longer names the net of U2.9 (CLK1)
- net CLK1: now also U6.11 (C); no longer U6.3 (C)
- net CLK2: no longer names the net of U2.6 (CLK2)
- net CLK2: now also U1.5
- new net: U6.12 (D), U6.5 (Q)
- new net: U1.4, U3.8 (~{Q})
- new net APURESET: U4.3 (RA4)
Other:
- moved on the sheet: C2, C5, C6, J1, U5, U6A, U6B, U6C

Commit message: back to old style
Parts:
- added U7: ICE5LP1K-SG48, Package_DFN_QFN:QFN-48-1EP_7x7mm_P0.5mm_EP5.6x5.6mm, symbol FPGA_Lattice:ICE5LP1K-SG48
Connections:
- new net: U7.30 (VCC), U7.5 (VCC)

Commit message: new stuff
Parts:
- added R74: 1K, Resistor_SMD:R_0603_1608Metric, symbol Device:R
- added SW1: RESET SWITCH, symbol Switch:SW_DPST_x2
Connections:
- new net RESET: R74.2
Changed lines of the file:
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@@
   (junction (at 74.93 35.56) (diameter 0) (color 0 0 0 0)
   )
+  (junction (at 379.095 15.24) (diameter 0) (color 0 0 0 0)
+  )
   (junction (at 267.97 64.77) (diameter 0) (color 0 0 0 0)
   )
@@
   (junction (at 121.92 87.63) (diameter 0) (color 0 0 0 0)
   )
+  (junction (at 379.095 -1.905) (diameter 0) (color 0 0 0 0)
+  )
   (junction (at 168.91 39.37) (diameter 0) (color 0 0 0 0)
   )
@@
   (junction (at 74.93 57.15) (diameter 0) (color 0 0 0 0)
   )
+  (junction (at 404.495 3.81) (diameter 0) (color 0 0 0 0)
+  )
   (junction (at 100.33 81.28) (diameter 0) (color 0 0 0 0)
   )
@@
   (junction (at 256.54 123.19) (diameter 0) (color 0 0 0 0)
   )
+  (junction (at 404.495 10.795) (diameter 0) (color 0 0 0 0)
+  )
+  (wire (pts (xy 398.145 10.795) (xy 404.495 10.795))
+    (stroke (width 0) (type default))
+  )
   (wire (pts (xy 256.54 102.87) (xy 256.54 109.22))
     (stroke (width 0) (type default))
@@
     (stroke (width 0) (type default))
   )
+  (wire (pts (xy 379.095 15.24) (xy 379.095 -1.905))
+    (stroke (width 0) (type default))
+  )
   (wire (pts (xy 223.52 80.01) (xy 234.95 80.01))
     (stroke (width 0) (type default))
   )
+  (wire (pts (xy 413.385 10.795) (xy 411.48 10.795))
+    (stroke (width 0) (type default))
+  )
   (wire (pts (xy 234.95 72.39) (xy 250.19 72.39))
     (stroke (width 0) (type default))
   )
+  (wire (pts (xy 374.65 17.145) (xy 379.095 17.145))
+    (stroke (width 0) (type default))
+  )
   (wire (pts (xy 176.53 59.69) (xy 167.64 59.69))
     (stroke (width 0) (type default))
@@
     (stroke (width 0) (type default))
   )
+  (wire (pts (xy 404.495 3.81) (xy 404.495 10.795))
+    (stroke (width 0) (type default))
+  )
   (wire (pts (xy 222.25 87.63) (xy 234.95 87.63))
     (stroke (width 0) (type default))
   )
+  (wire (pts (xy 404.495 15.24) (xy 379.095 15.24))
+    (stroke (width 0) (type default))
+  )
   (wire (pts (xy 105.41 80.01) (xy 105.41 81.28))
     (stroke (width 0) (type default))
@@
     (stroke (width 0) (type default))
   )
+  (wire (pts (xy 404.495 10.795) (xy 404.495 15.24))
+    (stroke (width 0) (type default))
+  )
   (wire (pts (xy 251.46 64.77) (xy 250.19 64.77))
     (stroke (width 0) (type default))
@@
     (stroke (width 0) (type default))
   )
+  (wire (pts (xy 392.43 -3.175) (xy 403.225 -3.175))
+    (stroke (width 0) (type default))
+  )
   (wire (pts (xy 77.47 54.61) (xy 83.82 54.61))
     (stroke (width 0) (type default))
@@
     (stroke (width 0) (type default))
   )
+  (wire (pts (xy 404.495 3.81) (xy 413.385 3.81))
+    (stroke (width 0) (type default))
+  )
   (wire (pts (xy 85.09 100.33) (xy 90.17 100.33))
     (stroke (width 0) (type default))
@@
     (stroke (width 0) (type default))
   )
+  (wire (pts (xy 394.97 3.81) (xy 394.97 -0.635))
+    (stroke (width 0) (type default))
+  )
+  (wire (pts (xy 379.095 17.145) (xy 379.095 15.24))
+    (stroke (width 0) (type default))
+  )
+  (wire (pts (xy 361.95 -1.905) (xy 365.76 -1.905))
+    (stroke (width 0) (type default))
+  )
   (wire (pts (xy 105.41 81.28) (xy 107.95 81.28))
     (stroke (width 0) (type default))
@@
     (stroke (width 0) (type default))
   )
+  (wire (pts (xy 402.59 3.81) (xy 404.495 3.81))
+    (stroke (width 0) (type default))
+  )
   (wire (pts (xy 176.53 29.21) (xy 176.53 31.75))
     (stroke (width 0) (type default))
@@
     (stroke (width 0) (type default))
   )
+  (wire (pts (xy 375.285 -1.905) (xy 379.095 -1.905))
+    (stroke (width 0) (type default))
+  )
   (wire (pts (xy 99.06 33.02) (xy 99.06 39.37))
     (stroke (width 0) (type default))
@@
     (stroke (width 0) (type default))
   )
+  (wire (pts (xy 394.97 -0.635) (xy 392.43 -0.635))
+    (stroke (width 0) (type default))
+  )
   (wire (pts (xy 267.97 64.77) (xy 266.7 64.77))
     (stroke (width 0) (type default))
@@
     (stroke (width 0) (type default))
   )
+  (wire (pts (xy 411.48 10.795) (xy 411.48 19.05))
+    (stroke (width 0) (type default))
+  )
   (wire (pts (xy 74.93 110.49) (xy 90.17 110.49))
     (stroke (width 0) (type default))
   )
+  (wire (pts (xy 379.095 -1.905) (xy 382.905 -1.905))
+    (stroke (width 0) (type default))
+  )
   (wire (pts (xy 74.93 57.15) (xy 74.93 110.49))
     (stroke (width 0) (type default))
@@
     (stroke (width 0) (type default))
   )
+  (wire (pts (xy 374.65 19.05) (xy 411.48 19.05))
+    (stroke (width 0) (type default))
+  )
   (wire (pts (xy 224.79 77.47) (xy 234.95 77.47))
     (stroke (width 0) (type default))
@@
     (stroke (width 0) (type default))
   )
+  (text_box "FPGA"
+    (at 365.125 15.24 0) (size 9.525 5.08)
+    (stroke (width 0) (type default))
+    (fill (type color) (color 255 255 194 1))
+    (effects (font (size 1.27 1.27)))
+  )
+  (text_box "DSP/SMP"
+    (at 413.385 8.255 0) (size 9.525 5.08)
+    (stroke (width 0) (type default))
+    (fill (type color) (color 255 255 194 1))
+    (effects (font (size 1.27 1.27)))
+  )
+  (text_box "PPU2"
+    (at 382.905 -4.445 0) (size 9.525 5.08)
+    (stroke (width 0) (type default))
+    (fill (type color) (color 255 255 194 1))
+    (effects (font (size 1.27 1.27)))
+  )
+  (text_box "CPU"
+    (at 413.385 1.27 0) (size 9.525 5.08)
+    (stroke (width 0) (type default))
+    (fill (type color) (color 255 255 194 1))
+    (effects (font (size 1.27 1.27)))
+  )
+  (text_box "PPU1"
+    (at 403.225 -5.08 0) (size 9.525 5.08)
+    (stroke (width 0) (type default))
+    (fill (type color) (color 255 255 194 1))
+    (effects (font (size 1.27 1.27)))
+  )
+  (text_box "CIC"
+    (at 365.76 -4.445 0) (size 9.525 5.08)
+    (stroke (width 0) (type default))
+    (fill (type color) (color 255 255 194 1))
+    (effects (font (size 1.27 1.27)))
+  )
+  (text_box "PST529"
+    (at 388.62 8.255 0) (size 9.525 5.08)
+    (stroke (width 0) (type default))
+    (fill (type color) (color 255 255 194 1))
+    (effects (font (size 1.27 1.27)))
+  )
   (text "Jumper MCLR to 3.3v when programmed\n" (at 34.29 40.64 0)
     (effects (font (size 1.27 1.27)) (justify left bottom))
@@
     (effects (font (size 1.27 1.27)) (justify left bottom))
   )
+  (label "RESOUT1" (at 403.225 3.81 0) (fields_autoplaced)
+    (effects (font (size 1.27 1.27)) (justify left bottom))
+  )
   (label "SMPWR" (at 135.89 46.99 90) (fields_autoplaced)
     (effects (font (size 1.27 1.27)) (justify left bottom))
   )
+  (label "RESET" (at 375.92 -1.905 0) (fields_autoplaced)
+    (effects (font (size 1.27 1.27)) (justify left bottom))
+  )
   (label "I2C_SDA" (at 224.79 74.93 0) (fields_autoplaced)
+    (effects (font (size 1.27 1.27)) (justify left bottom))
+  )
+  (label "RESOUT0" (at 393.7 -3.175 0) (fields_autoplaced)
     (effects (font (size 1.27 1.27)) (justify left bottom))
   )
@@
         (path "/e6d4ff55-0377-40c6-85e0-bfd48c6c6235"
           (reference "R1") (unit 1)
+        )
+      )
+    )
+  )
+  (symbol (lib_id "Switch:SW_DPST_x2") (at 356.87 -1.905 0) (unit 1)
+    (in_bom yes) (on_board yes) (dnp no)
+    (property "Reference" "SW1" (at 356.87 -5.715 0)
+      (effects (font (size 1.27 1.27)) hide)
+    )
+    (property "Value" "RESET SWITCH" (at 356.87 0.635 0)
+      (effects (font (size 1.27 1.27)))
+    )
+    (property "Footprint" "" (at 356.87 -1.905 0)
+      (effects (font (size 1.27 1.27)) hide)
+    )
+    (property "Datasheet" "~" (at 356.87 -1.905 0)
+      (effects (font (size 1.27 1.27)) hide)
+    )
+    (pin "1")
+    (pin "2")
+    (pin "3")
+    (pin "4")
+    (instances
+      (project "TAStable"
+        (path "/e6d4ff55-0377-40c6-85e0-bfd48c6c6235"
+          (reference "SW1") (unit 1)
         )
       )
@@
         )
       )
+    )
+  )
+  (symbol (lib_id "Device:R") (at 398.78 3.81 90) (mirror x) (unit 1)
+    (in_bom yes) (on_board yes) (dnp no)
+    (property "Reference" "R74" (at 396.24 6.35 90)
+      (effects (font (size 1.27 1.27)) (justify left))
+    )
+    (property "Value" "1K" (at 404.495 6.35 90)
+      (effects (font (size 1.27 1.27)) (justify left))
+    )
+    (property "Footprint" "Resistor_SMD:R_0603_1608Metric" (at 398.78 2.032 90)
+      (effects (font (size 1.27 1.27)) hide)
+    )
+    (property "Datasheet" "~" (at 398.78 3.81 0)
+      (effects (font (size 1.27 1.27)) hide)
+    )
+    (pin "1")
+    (pin "2")
+    (instances
+      (project "TAStable"
+        (path "/e6d4ff55-0377-40c6-85e0-bfd48c6c6235"
+          (reference "R74") (unit 1)
+        )
+      )
