File: TAStable.kicad_pcb (KiCad board)
At the start: 2 copper layers, 26.8 x 16.5 mm, 18 parts, among them J1 IN/OUT, J2 ICSP, U1 74HCT1G04, U2 CS2300-CP, U3 74LVC1G14, U4 PIC16LF15313, U6 AZ1117-3.3

Commit message: fixes
Parts:
- removed C7: 1uF, Capacitor_SMD:C_0603_1608Metric
- added C9: 100nF, Capacitor_SMD:C_0603_1608Metric, F.Cu at (163.6, 108.5)
- added U5: AZ1117-3.3, Package_TO_SOT_SMD:SOT-89-3, F.Cu at (159.3, 92.2)
- added Y2: 25MHz, Crystal:Crystal_SMD_Abracon_ABM8G-4Pin_3.2x2.5mm, F.Cu at (148.8, 106.4)
- C2: value 100nF -> 1uF
- C5: value 1uF -> 22uF Tantalum; footprint Capacitor_SMD:C_0603_1608Metric -> Capacitor_SMD:C_1206_3216Metric
- C6: value 22uF Tantalum -> 100nF; footprint Capacitor_SMD:C_1206_3216Metric -> Capacitor_SMD:C_0603_1608Metric
- J1: value IN/OUT -> Conn_01x08; footprint Connector_PinHeader_2.54mm:PinHeader_1x06_P2.54mm_Horizontal -> Connector_PinHeader_2.54mm:PinHeader_1x08_P2.54mm_Vertical
- U2: value CS2300-CP -> Si5351A-B-GT
- U3: value 74LVC1G14 -> 74HCT1G04
- U6: value AZ1117-3.3 -> 74HCT74; footprint Package_TO_SOT_SMD:SOT-89-3 -> Package_SO:TSSOP-14_4.4x5mm_P0.65mm
- moved C2 36.5 mm to (163.8, 91.9), turned to -90 degrees
- moved U6 35.6 mm to (160.3, 98.8)
- moved C6 35.4 mm to (160.4, 102.4)
- moved C4 30.1 mm to (163.6, 105.4)
- moved C8 30.1 mm to (150.6, 102.1)
- moved U3 26.4 mm to (161.3, 108.5), turned to 0 degrees
- moved J1 26.1 mm to (167.1, 90.7)
- moved U4 25.7 mm to (150.6, 98.8), turned to 180 degrees
- moved U2 25.6 mm to (154.9, 107.2), turned to 0 degrees
- moved U1 24.8 mm to (161.3, 105.4), turned to 0 degrees
- moved C1 24.0 mm to (153.7, 104.6)
- moved C3 22.9 mm to (159.0, 107.4), turned to 90 degrees
- moved C5 18.2 mm to (155.4, 92.3)
- moved R3 17.5 mm to (149.9, 94.0)
- moved J2 14.5 mm to (107.9, 95.5)
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Connections:
- C1 pad 1: GND -> +3.3V
- C1 pad 2: Net-(U2-XTO) -> GND
- C2 pad 1: +3.3V -> +5V
- C5 pad 1: +5V -> +3.3V
- C6 pad 1: +3.3V -> +5V
- J1 pad 5: /21MHz_IN -> /RESET_IN
- J1 pad 6: /24MHz_OUT -> /RESET_OUT
- J2 pad 4: /ICSPDAT -> /RESET_IN
- R3 pad 2: Net-(U2-AD0/~{CS}) -> /RESET_IN
- U1 pad 2: Net-(U2-CLK_OUT) -> /CLK0
- U1 pad 4: /24MHz_OUT -> /21MHz_OUT
- U2 pad 10: /I2C_SDA -> /CLK0
- U2 pad 2: GND -> Net-(U2-XA)
- U2 pad 3: Net-(U2-CLK_OUT) -> Net-(U2-XB)
- U2 pad 4: unconnected-(U2-AUX_OUT-Pad4) -> /I2C_SCL
- U2 pad 5: Net-(U2-CLK_IN) -> /I2C_SDA
- U2 pad 6: Net-(U2-XTO) -> /CLK2
- U2 pad 7: GND -> +3.3V
- U2 pad 8: Net-(U2-AD0/~{CS}) -> GND
- U2 pad 9: /I2C_SCL -> /CLK1
- U3 pad 2: /21MHz_IN -> /CLK2
- U3 pad 4: Net-(U2-CLK_IN) -> /24MHz_OUT
- U3 pad 5: +3.3V -> +5V
- U4 pad 2: unconnected-(U4-RA5-Pad2) -> Net-(U4-RA5)
- U4 pad 3: unconnected-(U4-RA4-Pad3) -> Net-(U4-RA4)
- U4 pad 7: /ICSPDAT -> /RESET_IN
- U6 pad 1: GND -> Net-(U4-RA5)
- U6 pad 2: +3.3V -> Net-(U4-RA4)
- U6 pad 3: +5V -> /CLK1
Routing:
- net +3.3V: track 52.1 -> 0.00 mm
- net +5V: track 44.0 -> 0.00 mm
- net /I2C_SCL: track 38.7 -> 0.00 mm, vias 1 -> 0
- net GND: track 23.4 -> 0.00 mm, vias 14 -> 0
- net /I2C_SDA: track 23.1 -> 0.00 mm
- net /ICSPDAT: track 11.1 -> 0.00 mm, vias 1 -> 0
- net Net-(U2-CLK_OUT): track 10.0 -> 0.00 mm
- net /MCLR: track 9.90 -> 0.00 mm, vias 1 -> 0
- net Net-(U2-CLK_IN): track 6.21 -> 0.00 mm
- net /21MHz_IN: track 5.33 -> 0.00 mm
- net Net-(U2-AD0/~{CS}): track 4.75 -> 0.00 mm
- net /24MHz_OUT: track 3.78 -> 0.00 mm
- net Net-(U2-XTO): track 2.37 -> 0.00 mm
